File: nipper_inspector_circuit.kicad_pcb (KiCad board)
At the start: 2 copper layers, 18 parts, among them J1 Jack-DC, J2 Conn_01x04_Male, J3 Conn_01x03_Male, U1 LPC1768, U2 TB6612FNG

Commit message: 最新版
Parts:
- removed D2, D3, D4: LED, LED_THT:LED_D3.0mm
- removed H1, H2: MountingHole_Pad, MountingHole:MountingHole_2.2mm_M2_DIN965_Pad
- removed U2: TB6612FNG, MyFootprint:TB6612FNG
- added J4: Conn_01x02_Male, Connector_JST:JST_XH_B2B-XH-A_1x02_P2.50mm_Vertical, F.Cu at (104.1, 63.5)
- added J5: Conn_01x02_Male, Connector_JST:JST_XH_B2B-XH-A_1x02_P2.50mm_Vertical, F.Cu at (104.1, 71.1)
- added J6: Conn_01x02_Male, Connector_JST:JST_XH_B2B-XH-A_1x02_P2.50mm_Vertical, F.Cu at (104.1, 78.7)
- added J7: Conn_01x02_Male, Connector_JST:JST_XH_B2B-XH-A_1x02_P2.50mm_Vertical, F.Cu at (104.1, 86.4)
- added J8: Conn_01x02_Male, Connector_JST:JST_XH_B2B-XH-A_1x02_P2.50mm_Vertical, F.Cu at (104.1, 94.0)
- added J9: Conn_01x02_Male, Connector_JST:JST_XH_B2B-XH-A_1x02_P2.50mm_Vertical, F.Cu at (180.3, 43.1)
- added Q1: Q_NJFET_DGS, Package_TO_SOT_THT:TO-92L_Inline_Wide, F.Cu at (114.3, 40.6)
- added Q2: Q_NJFET_DGS, Package_TO_SOT_THT:TO-92L_Inline_Wide, F.Cu at (114.3, 48.3)
- added Q3: Q_NJFET_DGS, Package_TO_SOT_THT:TO-92L_Inline_Wide, F.Cu at (114.3, 55.9)
- added Q4: Q_NJFET_DGS, Package_TO_SOT_THT:TO-92L_Inline_Wide, F.Cu at (114.3, 63.5)
- added Q5: Q_NJFET_DGS, Package_TO_SOT_THT:TO-92L_Inline_Wide, F.Cu at (114.3, 71.1)
- added Q6: Q_NJFET_DGS, Package_TO_SOT_THT:TO-92L_Inline_Wide, F.Cu at (114.3, 78.7)
- added Q7: Q_NJFET_DGS, Package_TO_SOT_THT:TO-92L_Inline_Wide, F.Cu at (114.3, 86.4)
- added Q8: Q_NJFET_DGS, Package_TO_SOT_THT:TO-92L_Inline_Wide, F.Cu at (114.3, 94.0)
- added R10: 3.3k, Resistor_THT:R_Axial_DIN0207_L6.3mm_D2.5mm_P7.62mm_Horizontal, F.Cu at (119.4, 68.6)
- added R11: 100, Resistor_THT:R_Axial_DIN0207_L6.3mm_D2.5mm_P7.62mm_Horizontal, F.Cu at (127.0, 73.7)
- added R12: 3.3k, Resistor_THT:R_Axial_DIN0207_L6.3mm_D2.5mm_P7.62mm_Horizontal, F.Cu at (119.4, 76.2)
- added R13: 100, Resistor_THT:R_Axial_DIN0207_L6.3mm_D2.5mm_P7.62mm_Horizontal, F.Cu at (127.0, 81.3)
- added R14: 3.3k, Resistor_THT:R_Axial_DIN0207_L6.3mm_D2.5mm_P7.62mm_Horizontal, F.Cu at (119.4, 83.8)
- added R15: 100, Resistor_THT:R_Axial_DIN0207_L6.3mm_D2.5mm_P7.62mm_Horizontal, F.Cu at (127.0, 88.9)
- added R16: 3.3k, Resistor_THT:R_Axial_DIN0207_L6.3mm_D2.5mm_P7.62mm_Horizontal, F.Cu at (119.4, 91.4)
- added R17: 3.3k, Resistor_THT:R_Axial_DIN0207_L6.3mm_D2.5mm_P7.62mm_Horizontal, F.Cu at (172.7, 40.6)
- added R8: 3.3k, Resistor_THT:R_Axial_DIN0207_L6.3mm_D2.5mm_P7.62mm_Horizontal, F.Cu at (119.4, 61.0)
- added R9: 100, Resistor_THT:R_Axial_DIN0207_L6.3mm_D2.5mm_P7.62mm_Horizontal, F.Cu at (127.0, 66.0)
- added REF**: universal_B, MyFootprint:universal_B, F.Cu at (142.2, 63.5)
- J1: value Jack-DC -> Conn_01x02_Male
- J2: value Conn_01x04_Male -> Conn_01x02_Male; footprint Connector_JST:JST_XH_B4B-XH-A_1x04_P2.50mm_Vertical -> Connector_JST:JST_XH_B2B-XH-A_1x02_P2.50mm_Vertical
- J3: value Conn_01x03_Male -> Conn_01x02_Male; footprint Connector_JST:JST_XH_B3B-XH-A_1x03_P2.50mm_Vertical -> Connector_JST:JST_XH_B2B-XH-A_1x02_P2.50mm_Vertical
- R1, R3, R5, R7: value R -> 100
- R2, R4, R6: value R -> 3.3k
- moved J1 110.2 mm to (104.1, 40.6)
- moved R4 96.2 mm to (119.4, 45.7), turned to 0 degrees
- moved R2 82.7 mm to (119.4, 38.1), turned to 0 degrees
- moved J3 81.2 mm to (104.1, 55.9)
- moved R3 80.7 mm to (127.0, 43.2)
- moved J2 76.4 mm to (104.1, 48.3)
- moved R1 75.5 mm to (127.0, 35.6), turned to 180 degrees
- moved R6 74.7 mm to (119.4, 53.3)
- moved R7 71.3 mm to (127.0, 58.4), turned to 180 degrees
- moved R5 61.2 mm to (127.0, 50.8), turned to 180 degrees
- moved D1 53.4 mm to (172.7, 38.1), turned to 90 degrees
- moved U1 48.2 mm to (148.6, 62.2)
Connections:
- D1 pad 2: +BATT -> +12V
- J1 pad 1: +BATT -> Net-(J1-Pad1)
- J1 pad 2: GND -> +12V
- J2 pad 1: Enc_B -> Net-(J2-Pad1)
- J2 pad 2: Enc_A -> +12V
- J3 pad 1: Interruptor -> Net-(J3-Pad1)
- J3 pad 2: GND -> +12V
- R1 pad 1: GND -> sig0
- R1 pad 2: Net-(D1-Pad1) -> Net-(Q1-Pad2)
- R2 pad 1: GND -> Net-(Q1-Pad2)
- R2 pad 2: Net-(D2-Pad1) -> GND
- R3 pad 1: GND -> sig1
- R3 pad 2: Net-(D3-Pad1) -> Net-(Q2-Pad2)
- R4 pad 1: GND -> Net-(Q2-Pad2)
- R4 pad 2: Net-(D4-Pad1) -> GND
- R5 pad 1: Enc_A -> sig2
- R5 pad 2: VDD -> Net-(Q3-Pad2)
- R6 pad 1: Enc_B -> Net-(Q3-Pad2)
- R6 pad 2: VDD -> GND
- R7 pad 1: Interruptor -> sig3
- R7 pad 2: VDD -> Net-(Q4-Pad2)
- U1 pad 12: Net-(U1-Pad12) -> sig4
- U1 pad 15: Net-(U1-Pad15) -> sig5
- U1 pad 16: Enc_A -> Net-(U1-Pad16)
- U1 pad 17: Enc_B -> Net-(U1-Pad17)
- U1 pad 18: Interruptor -> sig6
- U1 pad 20: Net-(U1-Pad20) -> sig7
- U1 pad 21: PWM -> Net-(U1-Pad21)
- U1 pad 22: SIG_2 -> Net-(U1-Pad22)
- U1 pad 23: SIG_1 -> Net-(U1-Pad23)
- U1 pad 5: Net-(U1-Pad5) -> sig0
- U1 pad 6: Net-(U1-Pad6) -> sig1
- U1 pad 7: Net-(U1-Pad7) -> sig2
- U1 pad 9: Net-(U1-Pad9) -> sig3
Routing:
- net VDD: track 217.6 -> 0.00 mm, vias 12 -> 0
- net +12V: track 0.00 -> 170.2 mm
- net +BATT: track 58.0 -> 0.00 mm
- net Interruptor: track 48.3 -> 0.00 mm, vias 2 -> 0
- net Enc_A: track 38.1 -> 0.00 mm, vias 2 -> 0
- net SIG_2: track 33.0 -> 0.00 mm
- net Enc_B: track 33.0 -> 0.00 mm, vias 2 -> 0
- net PWM: track 27.9 -> 0.00 mm, vias 2 -> 0
- net SIG_1: track 22.9 -> 0.00 mm
- net sig0: track 0.00 -> 22.9 mm
- net sig1: track 0.00 -> 17.8 mm
- net MT_2: track 15.2 -> 0.00 mm
- net sig7: track 0.00 -> 12.7 mm
- net sig2: track 0.00 -> 12.7 mm
- net MT_1: track 12.3 -> 0.00 mm
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Other:
- net class Default added: clearance 0.2, trace_width 0.25, via_dia 0.8, via_drill 0.4
