File: nipper_inspector_circuit.sch (KiCad schematic (older format))
At the start: 18 parts, among them J1 Jack-DC, J2 Conn_01x04_Male, J3 Conn_01x03_Male, U1 LPC1768, U2 TB6612FNG

Commit message: 最新版
Parts:
- removed D2, D3, D4: LED, LED_THT:LED_D3.0mm, symbol Device:LED
- removed H1, H2: MountingHole_Pad, MountingHole:MountingHole_2.2mm_M2_DIN965_Pad, symbol Mechanical:MountingHole_Pad
- removed J1: Jack-DC, Connector_JST:JST_XH_B2B-XH-A_1x02_P2.50mm_Vertical, symbol Connector:Jack-DC
- removed J2: Conn_01x04_Male, Connector_JST:JST_XH_B4B-XH-A_1x04_P2.50mm_Vertical, symbol Connector:Conn_01x04_Male
- removed J3: Conn_01x03_Male, Connector_JST:JST_XH_B3B-XH-A_1x03_P2.50mm_Vertical, symbol Connector:Conn_01x03_Male
- removed U2: TB6612FNG, MyFootprint:TB6612FNG, symbol MyComponent:TB6612FNG
- added J1, J2, J3, J4, J5, J6, J7, J8, J9: Conn_01x02_Male, Connector_JST:JST_XH_B2B-XH-A_1x02_P2.50mm_Vertical, symbol Connector:Conn_01x02_Male
- added Q1, Q2, Q3, Q4, Q5, Q6, Q7, Q8: Q_NJFET_DGS, Package_TO_SOT_THT:TO-92L_Inline_Wide, symbol Device:Q_NJFET_DGS
- added R10, R12, R14, R16, R17, R8: 3.3k, Resistor_THT:R_Axial_DIN0207_L6.3mm_D2.5mm_P7.62mm_Horizontal, symbol Device:R
- added R11, R13, R15, R9: 100, Resistor_THT:R_Axial_DIN0207_L6.3mm_D2.5mm_P7.62mm_Horizontal, symbol Device:R
- R1, R3, R5, R7: value R -> 100
- R2, R4, R6: value R -> 3.3k
Connections:
- net labels added: +12V, sig0, sig1, sig2, sig3, sig4, sig5, sig6, sig7
- net labels removed: +BATT, Enc_A, Enc_B, Interruptor, MT_1, MT_2, PWM, SIG_1, SIG_2
- wire segments 80 -> 102
- no-connect marks 32 -> 27
Other:
- moved on the sheet: U1
